File: KiCad_and_Gerbers/Resonant_Converter_V1/Resonant_Converter_V1.kicad_sch (KiCad schematic)
At the start: 193 parts, among them IC1 MC78M12BDTG, IC3 MAX253CSA+, IC4 AMC1306M25QDWVRQ1, IC5 AMC1306M25QDWVRQ1, IC9 AMC1306M25QDWVRQ1, J1 Screw_Terminal_01x02, J3 Screw_Terminal_01x02, J4 Conn_01x05_Male, J5 Conn_01x02_Male, Q1 STF35N60DM2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

Commit message: Small mods to schematic
Parts:
- C47: value 100nF -> 2.2uF
- C74, C75: value 10uF -> 2.2uF
- R10, R21, R8: value 22R -> 5R
- R12, R20: value 680R -> 1K
- R22, R60, R61, R9: value 22R -> 10R
- R62: value 100K -> DNP
Connections:
- net D4_Sigma_Delta is gone; now on net D3_Sigma_Delta: IC9.6 (DOUT), U1.27 (PB1)
- net D3_Sigma_Delta: no longer U1.38 (PC7)
- no-connect marks 0 -> 1
Changed lines of the file:
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@@
   (junction (at 250.19 38.1) (diameter 0) (color 0 0 0 0)
   )
+  (no_connect (at 344.17 49.53))
   (wire (pts (xy 323.85 68.58) (xy 323.85 64.77))
     (stroke (width 0) (type default) (color 0 0 0 0))
@@
     (stroke (width 0) (type default) (color 0 0 0 0))
   )
-  (wire (pts (xy 199.39 250.19) (xy 218.44 250.19))
-    (stroke (width 0) (type default) (color 0 0 0 0))
-  )
   (wire (pts (xy 267.97 95.25) (xy 262.89 95.25))
     (stroke (width 0) (type default) (color 0 0 0 0))
@@
     )
   )
-  (global_label "D3_Sigma_Delta" (shape input) (at 199.39 250.19 180) (fields_autoplaced)
-    (effects (font (size 1.27 1.27)) (justify right))
-    (property "Intersheet References" "${INTERSHEET_REFS}" (id 0) (at 181.9468 250.1106 0)
-      (effects (font (size 1.27 1.27)) (justify right) hide)
-    )
-  )
   (global_label "B_H_HV" (shape input) (at 49.53 102.87 180) (fields_autoplaced)
     (effects (font (size 1.27 1.27)) (justify right))
@@
     )
   )
-  (global_label "D4_Sigma_Delta" (shape input) (at 317.5 245.11 180) (fields_autoplaced)
+  (global_label "D3_Sigma_Delta" (shape input) (at 317.5 245.11 180) (fields_autoplaced)
     (effects (font (size 1.27 1.27)) (justify right))
     (property "Intersheet References" "${INTERSHEET_REFS}" (id 0) (at 300.0568 245.0306 0)
@@
     )
   )
-  (global_label "D4_Sigma_Delta" (shape input) (at 255.27 234.95 0) (fields_autoplaced)
+  (global_label "D3_Sigma_Delta" (shape input) (at 255.27 234.95 0) (fields_autoplaced)
     (effects (font (size 1.27 1.27)) (justify left))
-    (property "Intersheet References" "${INTERSHEET_REFS}" (id 0) (at 272.7132 235.0294 0)
+    (property "Intersheet References" "${INTERSHEET_REFS}" (id 0) (at 272.7132 234.8706 0)
       (effects (font (size 1.27 1.27)) (justify left) hide)
     )
@@
       (effects (font (size 1.27 1.27)) (justify left))
     )
-    (property "Value" "22R" (id 1) (at 95.885 173.355 90)
+    (property "Value" "5R" (id 1) (at 95.885 173.355 90)
       (effects (font (size 1.27 1.27)) (justify left))
     )
@@
       (effects (font (size 1.27 1.27)) (justify left))
     )
-    (property "Value" "10uF" (id 1) (at 131.826 188.3922 0)
+    (property "Value" "2.2uF" (id 1) (at 131.826 188.3922 0)
       (effects (font (size 1.27 1.27)) (justify left))
     )
@@
     (in_bom yes) (on_board yes) (fields_autoplaced)
     (property "Reference" "R20" (id 0) (at 372.11 197.2142 90))
-    (property "Value" "680R" (id 1) (at 372.11 199.7511 90))
+    (property "Value" "1K" (id 1) (at 372.11 199.7511 90))
     (property "Footprint" "Resistor_SMD:R_0603_1608Metric" (id 2) (at 372.11 203.708 90)
       (effects (font (size 1.27 1.27)) hide)
@@
       (effects (font (size 1.27 1.27)) (justify left))
     )
-    (property "Value" "10uF" (id 1) (at 157.226 188.3922 0)
+    (property "Value" "2.2uF" (id 1) (at 157.226 188.3922 0)
       (effects (font (size 1.27 1.27)) (justify left))
     )
@@
       (effects (font (size 1.27 1.27)) (justify left))
     )
-    (property "Value" "22R" (id 1) (at 175.26 158.75 90)
+    (property "Value" "10R" (id 1) (at 175.26 158.75 90)
       (effects (font (size 1.27 1.27)) (justify left))
     )
@@
       (effects (font (size 1.27 1.27)) (justify left))
     )
-    (property "Value" "22R" (id 1) (at 182.88 158.75 90)
+    (property "Value" "10R" (id 1) (at 182.88 158.75 90)
       (effects (font (size 1.27 1.27)) (justify left))
     )
@@
       (effects (font (size 1.27 1.27)) (justify left))
     )
-    (property "Value" "22R" (id 1) (at 118.11 180.34 90)
+    (property "Value" "10R" (id 1) (at 118.11 180.34 90)
       (effects (font (size 1.27 1.27)) (justify left))
     )
@@
       (effects (font (size 1.27 1.27)) (justify left))
     )
-    (property "Value" "680R" (id 1) (at 378.968 199.8222 0)
+    (property "Value" "1K" (id 1) (at 378.968 199.8222 0)
       (effects (font (size 1.27 1.27)) (justify left))
     )
@@
       (effects (font (size 1.27 1.27)) (justify left))
     )
-    (property "Value" "100K" (id 1) (at 228.6 158.75 90)
+    (property "Value" "DNP" (id 1) (at 228.6 158.75 90)
       (effects (font (size 1.27 1.27)) (justify left))
     )
@@
       (effects (font (size 1.27 1.27)) (justify left))
     )
-    (property "Value" "100nF" (id 1) (at 216.281 161.7222 0)
+    (property "Value" "2.2uF" (id 1) (at 216.281 161.7222 0)
       (effects (font (size 1.27 1.27)) (justify left))
     )
@@
       (effects (font (size 1.27 1.27)) (justify left))
     )
-    (property "Value" "22R" (id 1) (at 118.11 172.72 90)
+    (property "Value" "10R" (id 1) (at 118.11 172.72 90)
       (effects (font (size 1.27 1.27)) (justify left))
     )
@@
       (effects (font (size 1.27 1.27)) (justify left))
     )
-    (property "Value" "22R" (id 1) (at 95.885 158.115 90)
+    (property "Value" "5R" (id 1) (at 95.885 158.115 90)
       (effects (font (size 1.27 1.27)) (justify left))
     )
@@
       (effects (font (size 1.27 1.27)) (justify left))
     )
-    (property "Value" "22R" (id 1) (at 95.885 165.735 90)
+    (property "Value" "5R" (id 1) (at 95.885 165.735 90)
       (effects (font (size 1.27 1.27)) (justify left))
     )
@@
     )
     (path "/da5273db-da5b-4fee-9bd0-f3982cecaeb8"
-      (reference "C47") (unit 1) (value "100nF") (footprint "Capacitor_SMD:C_0603_1608Metric")
+      (reference "C47") (unit 1) (value "2.2uF") (footprint "Capacitor_SMD:C_0603_1608Metric")
     )
     (path "/750cbd04-57e3-428c-9638-2bb44a1dd570"
@@
     )
     (path "/296111a0-ec60-4d3a-9cac-a894157b3ca8"
-      (reference "C74") (unit 1) (value "10uF") (footprint "Capacitor_SMD:C_0603_1608Metric")
+      (reference "C74") (unit 1) (value "2.2uF") (footprint "Capacitor_SMD:C_0603_1608Metric")
     )
     (path "/3ca9e297-1c2e-45fc-a544-ba164d214aa3"
-      (reference "C75") (unit 1) (value "10uF") (footprint "Capacitor_SMD:C_0603_1608Metric")
+      (reference "C75") (unit 1) (value "2.2uF") (footprint "Capacitor_SMD:C_0603_1608Metric")
     )
     (path "/32234eca-425a-48bf-bb28-a233b5e0ec45"
@@
     )
     (path "/f1966a91-add4-454f-b3bf-cb573be7d1ea"
-      (reference "R8") (unit 1) (value "22R") (footprint "Resistor_SMD:R_0805_2012Metric")
+      (reference "R8") (unit 1) (value "5R") (footprint "Resistor_SMD:R_0805_2012Metric")
     )
     (path "/e934b840-6286-486b-88b3-db54c5874c9f"
-      (reference "R9") (unit 1) (value "22R") (footprint "Resistor_SMD:R_0805_2012Metric")
+      (reference "R9") (unit 1) (value "10R") (footprint "Resistor_SMD:R_0805_2012Metric")
     )
     (path "/ff8e213b-3f32-4c5c-a383-44196e6a006f"
-      (reference "R10") (unit 1) (value "22R") (footprint "Resistor_SMD:R_0805_2012Metric")
+      (reference "R10") (unit 1) (value "5R") (footprint "Resistor_SMD:R_0805_2012Metric")
     )
     (path "/2f906c36-ccf6-41d8-86e3-61e97adaf634"
@@
     )
     (path "/cd057c0f-6174-421c-aec0-3d379fe5d3d7"
-      (reference "R12") (unit 1) (value "680R") (footprint "Resistor_SMD:R_0603_1608Metric")
+      (reference "R12") (unit 1) (value "1K") (footprint "Resistor_SMD:R_0603_1608Metric")
     )
     (path "/a55fc58a-fb49-4b43-9786-4ecbc1956135"
@@
     )
     (path "/3880546d-e912-45e8-a40c-007e120a63c9"
-      (reference "R20") (unit 1) (value "680R") (footprint "Resistor_SMD:R_0603_1608Metric")
+      (reference "R20") (unit 1) (value "1K") (footprint "Resistor_SMD:R_0603_1608Metric")
     )
     (path "/16508d5d-d3c6-4a0e-a493-a5503e545525"
-      (reference "R21") (unit 1) (value "22R") (footprint "Resistor_SMD:R_0805_2012Metric")
+      (reference "R21") (unit 1) (value "5R") (footprint "Resistor_SMD:R_0805_2012Metric")
     )
     (path "/a231238c-571c-485e-b10a-d4dc586c5899"
-      (reference "R22") (unit 1) (value "22R") (footprint "Resistor_SMD:R_0805_2012Metric")
+      (reference "R22") (unit 1) (value "10R") (footprint "Resistor_SMD:R_0805_2012Metric")
     )
     (path "/86efbdf6-0f8d-4737-b345-78a928d1252f"
@@
     )
     (path "/650ff65c-7c26-405c-abe7-a6d4341ebed9"
-      (reference "R60") (unit 1) (value "22R") (footprint "Resistor_SMD:R_0805_2012Metric")
+      (reference "R60") (unit 1) (value "10R") (footprint "Resistor_SMD:R_0805_2012Metric")
     )
     (path "/8aefa31b-6656-480b-8b84-98fcb4e679cb"
-      (reference "R61") (unit 1) (value "22R") (footprint "Resistor_SMD:R_0805_2012Metric")
+      (reference "R61") (unit 1) (value "10R") (footprint "Resistor_SMD:R_0805_2012Metric")
     )
     (path "/da4c996c-77bd-4727-96e6-8233eca62fe2"
-      (reference "R62") (unit 1) (value "100K") (footprint "Resistor_SMD:R_0603_1608Metric")
+      (reference "R62") (unit 1) (value "DNP") (footprint "Resistor_SMD:R_0603_1608Metric")
     )
     (path "/1eacc8a9-30b0-4288-be32-2c09187912e8"
